Commit message: Added InverseDynamicsController example, still some problem in control loop

File: manipulation/models/eve/urdf/eve_7dof_arms_relative.urdf (robot description, URDF)
Before this commit: robot Eve, 96 links, 95 joints
Links:
- removed link qbhand_left_base_link
- removed link qbhand_left_index_distal_link
- removed link qbhand_left_index_distal_virtual_link
- removed link qbhand_left_index_knuckle_link
- removed link qbhand_left_index_middle_link
- removed link qbhand_left_index_middle_virtual_link
- removed link qbhand_left_index_proximal_link
- removed link qbhand_left_index_proximal_virtual_link
- removed link qbhand_left_little_distal_link
- removed link qbhand_left_little_distal_virtual_link
- removed link qbhand_left_little_knuckle_link
- removed link qbhand_left_little_middle_link
- removed link qbhand_left_little_middle_virtual_link
- removed link qbhand_left_little_proximal_link
- removed link qbhand_left_little_proximal_virtual_link
- removed link qbhand_left_middle_distal_link
- removed link qbhand_left_middle_distal_virtual_link
- removed link qbhand_left_middle_knuckle_link
- removed link qbhand_left_middle_middle_link
- removed link qbhand_left_middle_middle_virtual_link
- removed link qbhand_left_middle_proximal_link
- removed link qbhand_left_middle_proximal_virtual_link
- removed link qbhand_left_palm_link
- removed link qbhand_left_ring_distal_link
- removed link qbhand_left_ring_distal_virtual_link
- removed link qbhand_left_ring_knuckle_link
- removed link qbhand_left_ring_middle_link
- removed link qbhand_left_ring_middle_virtual_link
- removed link qbhand_left_ring_proximal_link
- removed link qbhand_left_ring_proximal_virtual_link
- removed link qbhand_left_tendon_virtual_link
- removed link qbhand_left_thumb_distal_link
- removed link qbhand_left_thumb_distal_virtual_link
- removed link qbhand_left_thumb_knuckle_link
- removed link qbhand_left_thumb_proximal_link
- removed link qbhand_left_thumb_proximal_virtual_link
- removed link qbhand_right_base_link
- removed link qbhand_right_index_distal_link
- removed link qbhand_right_index_distal_virtual_link
- removed link qbhand_right_index_knuckle_link
- removed link qbhand_right_index_middle_link
- removed link qbhand_right_index_middle_virtual_link
- removed link qbhand_right_index_proximal_link
- removed link qbhand_right_index_proximal_virtual_link
- removed link qbhand_right_little_distal_link
- removed link qbhand_right_little_distal_virtual_link
- removed link qbhand_right_little_knuckle_link
- removed link qbhand_right_little_middle_link
- removed link qbhand_right_little_middle_virtual_link
- removed link qbhand_right_little_proximal_link
- removed link qbhand_right_little_proximal_virtual_link
- removed link qbhand_right_middle_distal_link
- removed link qbhand_right_middle_distal_virtual_link
- removed link qbhand_right_middle_knuckle_link
- removed link qbhand_right_middle_middle_link
- removed link qbhand_right_middle_middle_virtual_link
- removed link qbhand_right_middle_proximal_link
- removed link qbhand_right_middle_proximal_virtual_link
- removed link qbhand_right_palm_link
- removed link qbhand_right_ring_distal_link
- removed link qbhand_right_ring_distal_virtual_link
- removed link qbhand_right_ring_knuckle_link
- removed link qbhand_right_ring_middle_link
- removed link qbhand_right_ring_middle_virtual_link
- removed link qbhand_right_ring_proximal_link
- removed link qbhand_right_ring_proximal_virtual_link
- removed link qbhand_right_tendon_virtual_link
- removed link qbhand_right_thumb_distal_link
- removed link qbhand_right_thumb_distal_virtual_link
- removed link qbhand_right_thumb_knuckle_link
- removed link qbhand_right_thumb_proximal_link
- removed link qbhand_right_thumb_proximal_virtual_link
- link base: geometry collision box size=.4 .15 .6; collision sphere radius=0.05
- link head: geometry collision sphere radius=0.12; visual mesh filename=../meshes/head.obj scale=1 1 1
- link l_elbow: geometry collision sphere radius=0.07; visual mesh filename=../meshes/7dof_elbow.obj scale=1 1 1
- link l_palm: geometry collision sphere radius=0.05; visual mesh filename=../meshes/7dof_palm.obj scale=1 1 1
- link l_wheel: geometry collision cylinder length=0.02 radius=0.14; visual mesh filename=../meshes/wheel.obj scale=1 1 1
- link pelvis: geometry collision sphere radius=0.12; visual mesh filename=../meshes/7dof_torso.obj scale=1 1 1
- link r_elbow: geometry collision sphere radius=0.07; visual mesh filename=../meshes/7dof_elbow.obj scale=1 1 1
- link r_palm: geometry collision sphere radius=0.05; visual mesh filename=../meshes/7dof_palm.obj scale=1 1 1
- link r_wheel: geometry collision cylinder length=0.02 radius=0.14; visual mesh filename=../meshes/wheel.obj scale=1 1 1
Joints:
- removed joint qbhand_left_base_fixed_joint
- removed joint qbhand_left_index_distal_joint
- removed joint qbhand_left_index_distal_virtual_joint
- removed joint qbhand_left_index_knuckle_joint
- removed joint qbhand_left_index_middle_joint
- removed joint qbhand_left_index_middle_virtual_joint
- removed joint qbhand_left_index_proximal_joint
- removed joint qbhand_left_index_proximal_virtual_joint
- removed joint qbhand_left_little_distal_joint
- removed joint qbhand_left_little_distal_virtual_joint
- removed joint qbhand_left_little_knuckle_joint
- removed joint qbhand_left_little_middle_joint
- removed joint qbhand_left_little_middle_virtual_joint
- removed joint qbhand_left_little_proximal_joint
- removed joint qbhand_left_little_proximal_virtual_joint
- removed joint qbhand_left_middle_distal_joint
- removed joint qbhand_left_middle_distal_virtual_joint
- removed joint qbhand_left_middle_knuckle_joint
- removed joint qbhand_left_middle_middle_joint
- removed joint qbhand_left_middle_middle_virtual_joint
- removed joint qbhand_left_middle_proximal_joint
- removed joint qbhand_left_middle_proximal_virtual_joint
- removed joint qbhand_left_palm_fixed_joint
- removed joint qbhand_left_ring_distal_joint
- removed joint qbhand_left_ring_distal_virtual_joint
- removed joint qbhand_left_ring_knuckle_joint
- removed joint qbhand_left_ring_middle_joint
- removed joint qbhand_left_ring_middle_virtual_joint
- removed joint qbhand_left_ring_proximal_joint
- removed joint qbhand_left_ring_proximal_virtual_joint
- removed joint qbhand_left_synergy_joint
- removed joint qbhand_left_thumb_distal_joint
- removed joint qbhand_left_thumb_distal_virtual_joint
- removed joint qbhand_left_thumb_knuckle_joint
- removed joint qbhand_left_thumb_proximal_joint
- removed joint qbhand_left_thumb_proximal_virtual_joint
- removed joint qbhand_right_base_fixed_joint
- removed joint qbhand_right_index_distal_joint
- removed joint qbhand_right_index_distal_virtual_joint
- removed joint qbhand_right_index_knuckle_joint
- removed joint qbhand_right_index_middle_joint
- removed joint qbhand_right_index_middle_virtual_joint
- removed joint qbhand_right_index_proximal_joint
- removed joint qbhand_right_index_proximal_virtual_joint
- removed joint qbhand_right_little_distal_joint
- removed joint qbhand_right_little_distal_virtual_joint
- removed joint qbhand_right_little_knuckle_joint
- removed joint qbhand_right_little_middle_joint
- removed joint qbhand_right_little_middle_virtual_joint
- removed joint qbhand_right_little_proximal_joint
- removed joint qbhand_right_little_proximal_virtual_joint
- removed joint qbhand_right_middle_distal_joint
- removed joint qbhand_right_middle_distal_virtual_joint
- removed joint qbhand_right_middle_knuckle_joint
- removed joint qbhand_right_middle_middle_joint
- removed joint qbhand_right_middle_middle_virtual_joint
- removed joint qbhand_right_middle_proximal_joint
- removed joint qbhand_right_middle_proximal_virtual_joint
- removed joint qbhand_right_palm_fixed_joint
- removed joint qbhand_right_ring_distal_joint
- removed joint qbhand_right_ring_distal_virtual_joint
- removed joint qbhand_right_ring_knuckle_joint
- removed joint qbhand_right_ring_middle_joint
- removed joint qbhand_right_ring_middle_virtual_joint
- removed joint qbhand_right_ring_proximal_joint
- removed joint qbhand_right_ring_proximal_virtual_joint
- removed joint qbhand_right_synergy_joint
- removed joint qbhand_right_thumb_distal_joint
- removed joint qbhand_right_thumb_distal_virtual_joint
- removed joint qbhand_right_thumb_knuckle_joint
- removed joint qbhand_right_thumb_proximal_joint
- removed joint qbhand_right_thumb_proximal_virtual_joint

File: manipulation/models/eve/urdf/eve_7dof_arms_relative_no_hand_base.urdf (robot description, URDF)
Before this commit: robot Eve, 24 links, 23 joints
Links:
- link abdomen: geometry visual mesh filename=package://eve/meshes/abdomen.obj scale=1 1 1
- link ankle_y_link: geometry visual mesh filename=package://eve/meshes/ankle.obj scale=1 1 1
- link base: geometry collision box size=.4 .15 .6; collision sphere radius=0.05
- link hip_x_link: geometry visual mesh filename=package://eve/meshes/hip.obj scale=1 1 1
- link l_wheel: geometry collision cylinder length=0.02 radius=0.14; visual mesh filename=package://eve/meshes/wheel.obj scale=1 1 1
- link pelvis: geometry collision sphere radius=0.12; visual mesh filename=package://eve/meshes/7dof_torso.obj scale=1 1 1
- link r_wheel: geometry collision cylinder length=0.02 radius=0.14; visual mesh filename=package://eve/meshes/wheel.obj scale=1 1 1
- link shin: geometry visual mesh filename=package://eve/meshes/shin.obj scale=1 1 1
- link thigh: geometry visual mesh filename=package://eve/meshes/thigh.obj scale=1 1 1
Joints:
- joint j_ankle_x: axis 1.0 0.0 0.0 -> -1.0 0.0 0.0; child base -> ankle_y_link; parent ankle_y_link -> base
- joint j_ankle_y: axis 0.0 1.0 0.0 -> 0.0 -1.0 0.0; child ankle_y_link -> shin; origin xyz=0.0 0.0 -0.38 rpy=0.0 0.0 0.0 -> xyz=0.0 0.0 0.0 rpy=0.0 0.0 0.0; parent shin -> ankle_y_link
- joint j_hip_x: axis 1.0 0.0 0.0 -> -1.0 0.0 0.0; child hip_x_link -> abdomen; parent abdomen -> hip_x_link
- joint j_hip_y: axis 0.0 1.0 0.0 -> 0.0 -1.0 0.0; child thigh -> hip_x_link; origin xyz=0.0 0.0 0.0 rpy=0.0 0.0 0.0 -> xyz=0.0 0.0 0.4 rpy=0.0 0.0 0.0; parent hip_x_link -> thigh
- joint j_hip_z: axis 0.0 0.0 1.0 -> 0.0 0.0 -1.0; child abdomen -> pelvis; parent pelvis -> abdomen
- joint j_knee_y: axis 0.0 1.0 0.0 -> 0.0 -1.0 0.0; child shin -> thigh; origin xyz=0.0 0.0 -0.4 rpy=0.0 0.0 0.0 -> xyz=0.0 0.0 0.38 rpy=0.0 0.0 0.0; parent thigh -> shin
