Commit message: added sdf, the numbering problem of tree branch model seems still exist

File: manipulation/models/eve/urdf/eve_7dof_arms_relative_base_no_collision.urdf (robot description, URDF)
Before this commit: robot Eve_base, 5 links, 4 joints
Links:
- added link abdomen, mass 3.4381772; visual mesh filename=package://eve/meshes/abdomen.obj scale=1 1 1
- added link head, mass 2.355; visual mesh filename=../meshes/head.obj scale=1 1 1
- added link hip_x_link, mass 2.868669; visual mesh filename=package://eve/meshes/hip.obj scale=1 1 1
- added link l_elbow, mass 0.46261553; visual mesh filename=../meshes/7dof_elbow.obj scale=1 1 1
- added link l_lower_arm, mass 1.63933464; visual mesh filename=../meshes/7dof_forearm.obj scale=1 1 1
- added link l_palm, mass 0.1486378; visual mesh filename=../meshes/7dof_palm.obj scale=1 1 1
- added link l_scapula, mass 2.75566786; visual mesh filename=../meshes/7dof_scapula.obj scale=1 1 1
- added link l_shoulder, mass 0.70265653; visual mesh filename=../meshes/7dof_shoulder.obj scale=1 1 1
- added link l_upper_arm, mass 2.92531724; visual mesh filename=../meshes/7dof_upper_arm.obj scale=1 1 1
- added link l_wrist, mass 0.30363399; visual mesh filename=../meshes/7dof_wrist.obj scale=1 1 1
- added link pelvis, mass 10.11628645; visual mesh filename=package://eve/meshes/7dof_torso.obj scale=1 1 1
- added link r_elbow, mass 0.46261553; visual mesh filename=../meshes/7dof_elbow.obj scale=1 1 1
- added link r_lower_arm, mass 1.63933464; visual mesh filename=../meshes/7dof_forearm.obj scale=1 1 1
- added link r_palm, mass 0.1486378; visual mesh filename=../meshes/7dof_palm.obj scale=1 1 1
- added link r_scapula, mass 2.75566786; visual mesh filename=../meshes/7dof_scapula.obj scale=1 1 1
- added link r_shoulder, mass 0.70264272; visual mesh filename=../meshes/7dof_shoulder.obj scale=1 1 1
- added link r_upper_arm, mass 2.92531724; visual mesh filename=../meshes/7dof_upper_arm.obj scale=1 1 1
- added link r_wrist, mass 0.30363399; visual mesh filename=../meshes/7dof_wrist.obj scale=1 1 1
- added link thigh, mass 12.846698; visual mesh filename=package://eve/meshes/thigh.obj scale=1 1 1
Joints:
- added joint j_hip_x: type revolute, parent hip_x_link, child abdomen, origin xyz=0.0 0.0 0.0 rpy=0.0 0.0 0.0, axis 1.0 0.0 0.0, limit lower=-0.523599 upper=0.523599 effort=-1.0 velocity=1.0
- added joint j_hip_y: type revolute, parent thigh, child hip_x_link, origin xyz=0.0 0.0 0.4 rpy=0.0 0.0 0.0, axis 0.0 1.0 0.0, limit lower=-1.57 upper=0.174533 effort=-1.0 velocity=1.0
- added joint j_hip_z: type revolute, parent abdomen, child pelvis, origin xyz=0.0 0.0 0.0 rpy=0.0 0.0 0.0, axis 0.0 0.0 -1.0, limit lower=-1.0472 upper=1.0472 effort=-1.0 velocity=1.0
- added joint j_knee_y: type revolute, parent shin, child thigh, origin xyz=0.0 0.0 0.38 rpy=0.0 0.0 0.0, axis 0.0 1.0 0.0, limit lower=0.0 upper=2.583 effort=-1.0 velocity=1.0
- added joint j_l_elbow_y: type revolute, parent l_upper_arm, child l_elbow, origin xyz=0.0 0.0 -0.313989 rpy=0.0 0.0 0.0, axis 0.0 1.0 0.0, limit lower=-2.18166 upper=0.0 effort=-1.0 velocity=1.0
- added joint j_l_elbow_z: type revolute, parent l_elbow, child l_lower_arm, origin xyz=0.0 0.0 0.0 rpy=0.0 0.0 0.0, axis 0.0 0.0 1.0, limit lower=-1.5708 upper=0.7854 effort=-1.0 velocity=1.0
- added joint j_l_shoulder_x: type revolute, parent l_scapula, child l_shoulder, origin xyz=0.0 0.0 0.0 rpy=-0.253261563 0.0 0.0, axis 1.0 0.0 0.0, limit lower=-0.0872665 upper=2.0943951 effort=-1.0 velocity=1.0
- added joint j_l_shoulder_y: type revolute, parent pelvis, child l_scapula, origin xyz=0.010525 0.207221 0.545525 rpy=0.253261563 0.0 -0.261799, axis 0.0 1.0 0.0, limit lower=-2.4240878 upper=0.981049573 effort=-1.0 velocity=1.0
- added joint j_l_shoulder_z: type revolute, parent l_shoulder, child l_upper_arm, origin xyz=0.0 0.0 0.0 rpy=0.0 0.0 0.261799, axis 0.0 0.0 1.0, limit lower=-2.0943951 upper=-0.0872665 effort=-1.0 velocity=1.0
- added joint j_l_wrist_x: type revolute, parent l_wrist, child l_palm, origin xyz=0.0 0.0 0.0 rpy=0.0 0.0 0.0, axis 1.0 0.0 0.0, limit lower=-1.5708 upper=0.523599 effort=-1.0 velocity=1.0
- added joint j_l_wrist_y: type revolute, parent l_lower_arm, child l_wrist, origin xyz=0.0 0.0 -0.29285 rpy=0.0 0.0 0.0, axis 0.0 1.0 0.0, limit lower=-0.785398 upper=0.785398 effort=-1.0 velocity=1.0
- added joint j_neck_y: type revolute, parent pelvis, child head, origin xyz=-0.004458 0.0 0.680766 rpy=0.0 0.0 0.0, axis 0.0 1 0.0, limit lower=-0.0872664626 upper=0.698132 effort=-1.0 velocity=1.0
- added joint j_r_elbow_y: type revolute, parent r_upper_arm, child r_elbow, origin xyz=0.0 0.0 -0.313989 rpy=0.0 0.0 0.0, axis 0.0 1 0.0, limit lower=-2.18166 upper=0.0 effort=-1.0 velocity=1.0
- added joint j_r_elbow_z: type revolute, parent r_elbow, child r_lower_arm, origin xyz=0.0 0.0 0.0 rpy=0.0 0.0 0.0, axis 0.0 0.0 1, limit lower=-0.7854 upper=1.5708 effort=-1.0 velocity=1.0
- added joint j_r_shoulder_x: type revolute, parent r_scapula, child r_shoulder, origin xyz=0.0 0.0 0.0 rpy=0.253261563 0.0 0.0, axis 1.0 0.0 0.0, limit lower=-2.0943951 upper=0.0872665 effort=-1.0 velocity=1.0
- added joint j_r_shoulder_y: type revolute, parent pelvis, child r_scapula, origin xyz=0.010525 -0.207221 0.545525 rpy=-0.253261563 0.0 0.261799, axis 0.0 1.0 0.0, limit lower=-2.4240878 upper=0.981049573 effort=-1.0 velocity=1.0
- added joint j_r_shoulder_z: type revolute, parent r_shoulder, child r_upper_arm, origin xyz=0.0 0.0 0.0 rpy=0.0 0.0 -0.261799, axis 0.0 0.0 1.0, limit lower=0.0872665 upper=2.0943951 effort=-1.0 velocity=1.0
- added joint j_r_wrist_x: type revolute, parent r_wrist, child r_palm, origin xyz=0.0 0.0 0.0 rpy=0.0 0.0 0.0, axis 1 0.0 0.0, limit lower=-0.523599 upper=1.5708 effort=-1.0 velocity=1.0
- added joint j_r_wrist_y: type revolute, parent r_lower_arm, child r_wrist, origin xyz=0.0 0.0 -0.292850 rpy=0.0 0.0 0.0, axis 0.0 1 0.0, limit lower=-0.785398 upper=0.785398 effort=-1.0 velocity=1.0
