Commit message: Eve moves with torque applied on wheel while upper body balanced by InverseDynamicsController

File: manipulation/models/eve/urdf/eve_7dof_arms_relative_base_collision.urdf (robot description, URDF)
Before this commit: robot Eve_base, 24 links, 23 joints
Joints:
- joint j_l_wheel_y: type fixed -> revolute
- joint j_r_wheel_y: type fixed -> revolute
